File: terrarium-light.kicad_pcb (KiCad board)
At the start: 2 copper layers, 100 x 100 mm, 51 parts, among them J2 USB_C_Receptacle_USB2.0_16P, Q1 UMH3N, U1 CH340C, U2 TPS61169DCKR, U3 TPS61169DCKR, U4 LM1117S-3.3, U6 ESP32-S3-MINI-1

Commit message: re do
Parts:
- moved D18 30.8 mm to (110.0, 109.2)
- moved D10 24.0 mm to (75.0, 124.7), turned to 180 degrees
- moved D20 21.0 mm to (110.0, 140.0)
- moved D22 20.6 mm to (139.0, 140.0)
- moved D19 18.2 mm to (110.0, 124.6)
- moved D21 17.7 mm to (124.5, 140.0)
- moved D23 16.2 mm to (140.0, 124.6)
- moved D8 15.6 mm to (90.0, 124.7), turned to 180 degrees
- moved D9 15.6 mm to (90.0, 109.3), turned to 180 degrees
- moved D15 11.4 mm to (124.5, 93.9)
- moved D7 10.0 mm to (90.0, 140.1), turned to 180 degrees
- moved D17 9.62 mm to (124.5, 124.6)
- moved D11 9.27 mm to (75.0, 109.3), turned to 180 degrees
- moved D24 8.25 mm to (140.0, 109.2)
- moved D16 7.01 mm to (124.5, 109.2)
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Routing:
- net Net-(D1-A): track 0.00 -> 18.6 mm
- net Net-(D5-K): track 0.00 -> 15.9 mm
- net Net-(D6-K): track 0.00 -> 15.0 mm
- net Net-(D8-K): track 0.00 -> 13.1 mm
- net Net-(D7-K): track 0.00 -> 13.1 mm
- net Net-(D4-K): track 0.00 -> 13.1 mm
- net Net-(D3-K): track 0.00 -> 13.1 mm
- net Net-(D2-K): track 0.00 -> 13.1 mm
- net Net-(D19-K): track 0.00 -> 13.1 mm
- net Net-(D18-K): track 0.00 -> 13.1 mm
- net Net-(D16-K): track 0.00 -> 13.1 mm
- net Net-(D15-K): track 0.00 -> 13.1 mm
- net Net-(D11-K): track 0.00 -> 13.1 mm
- net Net-(D10-K): track 0.00 -> 13.1 mm
- net Net-(D1-K): track 0.00 -> 13.1 mm
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
Commit message: changes
Parts:
- moved C2 2.16 mm to (116.0, 81.8), turned to 0 degrees
- moved C4 2.15 mm to (76.0, 81.9), turned to 0 degrees
- moved R2 1.26 mm to (119.8, 82.2)
- moved C1 1.25 mm to (124.7, 79.3)
- moved U3 1.25 mm to (120.3, 79.8)
- moved C3 1.25 mm to (84.7, 79.3)
- moved R1 1.25 mm to (79.8, 82.2)
- moved U2 1.25 mm to (80.3, 79.8)
Routing:
- net Net-(D1-A): track 18.6 -> 15.5 mm
- net +5V: track 6.57 -> 9.19 mm
- net Net-(D26-K): track 0.00 -> 1.38 mm
- net Net-(D12-K): track 2.03 -> 1.39 mm
- net (no net): vias 0 -> 12

Commit message: LOTS OF MOVING
Parts:
- moved C7 112.0 mm to (81.5, 57.0), turned to 180 degrees
- moved R4 107.1 mm to (95.7, 59.9), turned to 180 degrees
- moved FB1 103.3 mm to (103.2, 62.4), turned to -90 degrees
- moved C5 102.8 mm to (80.6, 64.2), turned to 180 degrees
- moved R3 101.7 mm to (101.2, 60.8), turned to -90 degrees
- moved C9 95.6 mm to (101.3, 81.8)
- moved C8 93.4 mm to (96.2, 81.8), turned to 180 degrees
- moved C6 87.5 mm to (89.0, 57.7), turned to -90 degrees
- moved C11 83.8 mm to (104.3, 65.3)
- moved C10 81.8 mm to (104.3, 59.5)
- moved U1 15.0 mm to (86.3, 64.8)
- moved Q1 7.73 mm to (85.1, 55.7)
- moved D22 1.00 mm to (140.0, 140.1), turned to 180 degrees
- moved D21 0.10 mm to (124.5, 140.1), turned to 180 degrees
- moved D23 0.10 mm to (140.0, 124.7), turned to 180 degrees
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Routing:
- net +5V: track 9.19 -> 88.6 mm
- net Net-(D10-A): track 0.00 -> 26.6 mm
- net Net-(D26-K): track 1.38 -> 27.8 mm
- net Net-(D17-K): track 0.00 -> 26.3 mm
- net Net-(D14-K): track 0.00 -> 18.0 mm
- net Net-(D21-K): track 0.00 -> 16.4 mm
- net Net-(D20-K): track 0.00 -> 14.5 mm
- net Net-(D25-K): track 0.00 -> 13.1 mm
- net Net-(D24-K): track 0.00 -> 13.1 mm
- net Net-(D23-K): track 0.00 -> 13.1 mm
- net Net-(D22-K): track 0.00 -> 13.1 mm
- net Net-(D12-K): track 1.39 -> 13.6 mm
- net VBUS: track 0.00 -> 11.5 mm
- net +3.3V: track 0.00 -> 7.66 mm
- net Net-(D14-A): track 0.00 -> 7.55 mm
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
Commit message: big changes and lots of routing
Parts:
- moved C7 12.2 mm to (93.4, 59.5), turned to 0 degrees
- moved C5 11.3 mm to (90.4, 69.9), turned to -90 degrees
- moved C6 6.43 mm to (83.8, 61.5), turned to 0 degrees
- moved Q1 5.88 mm to (90.1, 58.8), turned to 90 degrees
- moved U1 4.77 mm to (91.0, 64.2), turned to 90 degrees
- moved R4 1.62 mm to (97.2, 59.5)
Routing:
- net /D+: track 2.71 -> 21.0 mm
- net /D-: track 2.74 -> 20.2 mm, vias 0 -> 2
- net /~{RTS}: track 0.00 -> 4.28 mm
- net /~{DTR}: track 0.00 -> 4.27 mm
- net /ESP_EN: track 0.00 -> 2.57 mm
- net Net-(J2-CC2): track 0.00 -> 2.21 mm
- net /ESP_IO0: track 0.00 -> 1.80 mm

Commit message: little more routing
Routing:
- net +3.3V: track 7.66 -> 89.8 mm, vias 0 -> 4
- net /ESP_EN: track 2.57 -> 35.8 mm
Changed lines of the file:
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@@
 		(tags "SOT-363 SC-70-6")
 		(property "Reference" "Q1"
-			(at 0 -2.25 270)
+			(at 0 -2.25 -90)
 			(layer "F.SilkS")
 			(effects
@@
 		)
 		(property "Value" "UMH3N"
-			(at -0.6 -6.3 270)
+			(at -0.6 -6.3 -90)
 			(layer "F.Fab")
 			(hide yes)
@@
 		)
 		(fp_text user "${REFERENCE}"
-			(at 0 0 360)
+			(at 0 0 0)
 			(layer "F.Fab")
 			(effects
@@
 		(tags "SOIC SO")
 		(property "Reference" "U1"
-			(at 0 -5.9 270)
+			(at 0 -5.9 -90)
 			(layer "F.SilkS")
 			(effects
@@
 		)
 		(property "Value" "CH340C"
-			(at -0.05 -7.635 270)
+			(at -0.05 -7.635 -90)
 			(layer "F.Fab")
 			(hide yes)
@@
 		)
 		(fp_text user "${REFERENCE}"
-			(at 0 0 270)
+			(at 0 0 -90)
 			(layer "F.Fab")
 			(effects
@@
 		(tags "capacitor handsolder")
 		(property "Reference" "C6"
-			(at 0 -1.68 360)
+			(at 0 -1.68 0)
 			(layer "F.SilkS")
 			(effects
@@
 		)
 		(property "Value" "0.1uF "
-			(at -4.6125 0 360)
+			(at -4.6125 0 0)
 			(layer "F.Fab")
 			(effects
@@
 		)
 		(fp_text user "${REFERENCE}"
-			(at 0 0 360)
+			(at 0 0 0)
 			(layer "F.Fab")
 			(effects
@@
 		(tags "capacitor handsolder")
 		(property "Reference" "C7"
-			(at -0.05 -1.85 360)
+			(at -0.05 -1.85 0)
 			(layer "F.SilkS")
 			(effects
@@
 		)
 		(property "Value" "1uF "
-			(at 2.8 -1.85 360)
+			(at 2.8 -1.85 0)
 			(layer "F.Fab")
 			(effects
@@
 		)
 		(fp_text user "${REFERENCE}"
-			(at 0 0 360)
+			(at 0 0 0)
 			(layer "F.Fab")
 			(effects
@@
 	)
 	(segment
+		(start 84.3325 52.8)
+		(end 58.3 52.8)
+		(width 0.4)
+		(layer "F.Cu")
+		(net 3)
+	)
+	(segment
+		(start 89.4225 57.89)
+		(end 84.3325 52.8)
+		(width 0.4)
+		(layer "F.Cu")
+		(net 3)
+	)
+	(segment
 		(start 58.3 52.8)
 		(end 57.05 54.05)
@@
 	)
 	(segment
+		(start 58.75 73.44)
+		(end 58.75 68.85)
+		(width 0.2)
+		(layer "F.Cu")
+		(net 13)
+	)
+	(segment
+		(start 92.78 73.31)
+		(end 92.78 70.54875)
+		(width 1)
+		(layer "F.Cu")
+		(net 13)
+	)
+	(segment
+		(start 85.87 60.52625)
+		(end 84.8825 61.51375)
+		(width 1)
+		(layer "F.Cu")
+		(net 13)
+	)
+	(segment
+		(start 85.87 59.84)
+		(end 85.87 60.52625)
+		(width 1)
+		(layer "F.Cu")
+		(net 13)
+	)
+	(segment
+		(start 100.2625 81.75)
+		(end 100.2625 81.1575)
+		(width 1)
+		(layer "F.Cu")
+		(net 13)
+	)
+	(segment
 		(start 86.5625 61.76375)
 		(end 85.1325 61.76375)
@@
 	)
 	(segment
+		(start 92.78 70.54875)
+		(end 91.1075 68.87625)
+		(width 1)
+		(layer "F.Cu")
+		(net 13)
+	)
+	(segment
+		(start 58.74 73.45)
+		(end 58.75 73.44)
+		(width 0.2)
+		(layer "F.Cu")
+		(net 13)
+	)
+	(segment
 		(start 90.3725 68.86625)
 		(end 90.3825 68.87625)
@@
 	)
 	(segment
+		(start 91.1075 68.87625)
+		(end 90.3825 68.87625)
+		(width 1)
+		(layer "F.Cu")
+		(net 13)
+	)
+	(segment
 		(start 85.1325 61.76375)
 		(end 84.8825 61.51375)
@@
 	)
 	(segment
+		(start 100.2625 81.1575)
+		(end 102.68 78.74)
+		(width 1)
+		(layer "F.Cu")
+		(net 13)
+	)
+	(segment
 		(start 100 85.35)
 		(end 100 82.0125)
@@
 		(net 13)
 	)
+	(via
+		(at 58.74 73.45)
+		(size 0.6)
+		(drill 0.3)
+		(layers "F.Cu" "B.Cu")
+		(net 13)
+	)
+	(via
+		(at 92.78 73.31)
+		(size 0.6)
+		(drill 0.3)
+		(layers "F.Cu" "B.Cu")
+		(net 13)
+	)
+	(via
+		(at 102.68 78.74)
+		(size 0.6)
+		(drill 0.3)
+		(layers "F.Cu" "B.Cu")
+		(net 13)
+	)
+	(via
+		(at 85.87 59.84)
+		(size 0.6)
+		(drill 0.3)
+		(layers "F.Cu" "B.Cu")
+		(net 13)
+	)
+	(segment
+		(start 93.45 73.45)
+		(end 58.74 73.45)
+		(width 1)
+		(layer "B.Cu")
+		(net 13)
+	)
+	(segment
+		(start 93.59 73.31)
+		(end 93.45 73.45)
+		(width 1)
+		(layer "B.Cu")
+		(net 13)
+	)
+	(segment
+		(start 102.68 78.74)
+		(end 97.25 73.31)
+		(width 1)
+		(layer "B.Cu")
+		(net 13)
+	)
+	(segment
+		(start 85.87 62.513503)
+		(end 85.87 59.84)
+		(width 1)
+		(layer "B.Cu")
+		(net 13)
+	)
+	(segment
+		(start 93.59 73.31)
+		(end 92.78 73.31)
+		(width 1)
+		(layer "B.Cu")
+		(net 13)
+	)
+	(segment
+		(start 97.25 73.31)
+		(end 96.666497 73.31)
+		(width 1)
+		(layer "B.Cu")
+		(net 13)
+	)
+	(segment
+		(start 97.25 73.31)
+		(end 93.59 73.31)
+		(width 1)
+		(layer "B.Cu")
+		(net 13)
+	)
+	(segment
+		(start 96.666497 73.31)
+		(end 85.87 62.513503)
+		(width 1)
+		(layer "B.Cu")
+		(net 13)
+	)

Commit message: changes
Parts:
- added J1: Conn_01x04_Pin, Connector_PinHeader_2.54mm:PinHeader_1x04_P2.54mm_Vertical, B.Cu at (114.0, 62.8)

Commit message: SO many changes
Parts:
- added SW1: RotaryEncoder_Switch_MP, Rotary_Encoder:RotaryEncoder_Alps_EC12E-Switch_Vertical_H20mm_CircularMountingHoles, B.Cu at (143.5, 57.0)
Routing:
- net Net-(D14-A): track 7.55 -> 9.15 mm
- net GND: vias 0 -> 10
- net (no net): vias 12 -> 0
- added copper zone on B.Cu, net GND
- added copper zone on F.Cu, net GND

Commit message: saving
Parts:
- added C12: 0.1uF, Capacitor_SMD:C_0805_2012Metric_Pad1.18x1.45mm_HandSolder, F.Cu at (122.0, 56.0)
- added C7: 0.1uF, Capacitor_SMD:C_0805_2012Metric_Pad1.18x1.45mm_HandSolder, F.Cu at (117.8, 60.3)
- added R5: 10k, Resistor_SMD:R_0805_2012Metric_Pad1.20x1.40mm_HandSolder, F.Cu at (126.0, 60.0)
- added R6: 1k, Resistor_SMD:R_0805_2012Metric_Pad1.20x1.40mm_HandSolder, F.Cu at (125.0, 57.0)
- added R7: 10k, Resistor_SMD:R_0805_2012Metric_Pad1.20x1.40mm_HandSolder, F.Cu at (146.0, 58.0)
- added R8: 10k, Resistor_SMD:R_0805_2012Metric_Pad1.20x1.40mm_HandSolder, F.Cu at (146.0, 62.0)
- moved U6 2.50 mm to (60.5, 64.3)
Connections:
- SW1 pad A: unconnected-(SW1-PadA) -> /EncoderA
- SW1 pad B: unconnected-(SW1-PadB) -> /EncoderB
- SW1 pad C: unconnected-(SW1-PadC) -> GND
- SW1 pad MP: unconnected-(SW1-PadMP) -> GND
- SW1 pad S1: unconnected-(SW1-PadS1) -> Net-(R5-Pad1)
- SW1 pad S2: unconnected-(SW1-PadS2) -> GND
Routing:
- net /ESP_EN: track 35.8 -> 38.3 mm
- net +3.3V: track 89.8 -> 87.3 mm
