File: terrarium-light.kicad_pcb (KiCad board)
At the start: 2 copper layers, 100 x 100 mm, 59 parts, among them J1 Conn_01x04_Pin, J2 USB_C_Receptacle_USB2.0_16P, Q1 UMH3N, SW1 RotaryEncoder_Switch_MP, U1 CH340C, U2 TPS61169DCKR, U3 TPS61169DCKR, U4 LM1117S-3.3, U6 ESP32-S3-MINI-1

Commit message: settings
Parts:
- removed the C7 at (93.4, 59.5)
- added kibuzzard-66CB9840: G***, kibuzzard-66CB9840, F.Cu at (142.8, 146.7)
- moved C6 17.8 mm to (91.4, 77.6)
- moved Q1 13.5 mm to (89.5, 72.3), turned to 180 degrees
- moved C5 10.3 mm to (100.6, 71.3), turned to 0 degrees
- moved U1 8.15 mm to (94.9, 71.4), turned to 180 degrees
- moved J1 3.22 mm to (117.2, 62.5)
- moved R7 2.62 mm to (144.1, 56.2)
- moved C7 2.55 mm to (120.1, 61.4), turned to 90 degrees
- moved C12 2.32 mm to (123.5, 54.2), turned to 180 degrees
- moved SW1 2.19 mm to (141.5, 56.1)
- moved R8 1.99 mm to (144.1, 61.4)
- moved R5 1.84 mm to (124.4, 59.1)
- moved R6 1.70 mm to (123.5, 56.2)
- moved R4 0.22 mm to (97.0, 59.5)
Routing:
- net +3.3V: track 87.3 -> 144.0 mm
- net /ESP_32_RX: track 0.00 -> 52.7 mm, vias 0 -> 2
- net /ESP_32_TX: track 0.00 -> 51.2 mm, vias 0 -> 2
- net /ESP_IO0: track 1.80 -> 35.5 mm
- net +5V: track 88.6 -> 81.9 mm
- net VBUS: track 11.5 -> 5.74 mm
- net Net-(R5-Pad1): track 0.00 -> 4.48 mm
- net /ESP_EN: track 38.3 -> 42.3 mm, vias 0 -> 2
- net /D-: track 20.2 -> 16.6 mm, vias 2 -> 0
- net /EncoderB: track 0.00 -> 3.14 mm
- net /EncoderA: track 0.00 -> 2.97 mm
- net /D+: track 21.0 -> 18.0 mm, vias 0 -> 2
- net /EncoderButton: track 0.00 -> 2.03 mm

Commit message: fixed
Routing:
- net /ESP_EN: track 42.3 -> 42.9 mm
Changed lines of the file:
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@@
 				(font
 					(size 0.001 0.001)
+					(thickness 0.15)
 				)
 			)
@@
 				(font
 					(size 0.001 0.001)
+					(thickness 0.15)
 				)
 			)
@@
 	)
 	(segment
-		(start 57.1 57.3)
-		(end 57.05 57.35)
+		(start 57.1 55.9)
+		(end 57.1 57.3)
 		(width 0.4)
 		(layer "F.Cu")
@@
 	)
 	(segment
-		(start 57.1 56.2)
-		(end 57.1 57.3)
+		(start 57.1 57.3)
+		(end 57.05 57.35)
 		(width 0.4)
 		(layer "F.Cu")
@@
 	)
 	(via
-		(at 57.1 56.2)
+		(at 57.1 55.9)
 		(size 0.5)
 		(drill 0.3)
@@
 	)
 	(segment
-		(start 70.5 73.5)
+		(start 57.1 55.9)
 		(end 57.1 60.1)
 		(width 0.4)
@@
 	)
 	(segment
-		(start 87.8 73.5)
+		(start 57.1 60.1)
 		(end 70.5 73.5)
 		(width 0.4)
@@
 	)
 	(segment
-		(start 57.1 60.1)
-		(end 57.1 56.2)
+		(start 70.5 73.5)
+		(end 87.8 73.5)
 		(width 0.4)
 		(layer "B.Cu")
