File: terrarium-light.kicad_sch (KiCad schematic)
At the start: 52 parts, among them J1 USB_C_Receptacle_USB2.0_14P, Q1 UMH3N, SW1 RotaryEncoder, U1 CH340C, U2 TPS61169DCKR, U3 TPS61169DCKR, U4 LM1117S-3.3, U5 ESP32-S3-MINI-1U

Commit message: found more parts and added them
Parts:
- removed C11: C_Polarized_Small, symbol Device:C_Polarized_Small
- removed J1: USB_C_Receptacle_USB2.0_14P, Connector_USB:USB_C_Receptacle_GCT_USB4105-xx-A_16P_TopMnt_Horizontal, symbol Connector:USB_C_Receptacle_USB2.0_14P
- added C11: 0.1uf, Capacitor_SMD:C_0805_2012Metric_Pad1.18x1.45mm_HandSolder, symbol Device:C_Small
- added J2: USB_C_Receptacle_USB2.0_16P, Connector_USB:USB_C_Receptacle_HCTL_HC-TYPE-C-16P-01A, symbol Connector:USB_C_Receptacle_USB2.0_16P
- C10, C5, C6, C7, C8, C9: footprint (none) -> Capacitor_SMD:C_0805_2012Metric_Pad1.18x1.45mm_HandSolder
- FB1: value FerriteBead_Small -> MI0805K400R-10
- R3, R4: footprint (none) -> Resistor_SMD:R_0805_2012Metric_Pad1.20x1.40mm_HandSolder
Connections:
- net +5V: now also FB1.2, C11.1
- net D+: now also J2.A6 (D+), J2.B6 (D+)
- net D-: now also J2.A7 (D-), J2.B7 (D-)
- net GND: now also C10.2, C11.2, J2.A1 (GND), J2.A12 (GND), J2.B1 (GND), J2.B12 (GND), J2.S1 (SHIELD)
- net VBUS: now reaches FB1.1
- net VBUS: now also C10.1, J2.A4 (VBUS), J2.A9 (VBUS), J2.B4 (VBUS), J2.B9 (VBUS)
- net at R3.1: now also J2.A5 (CC1)
- net at R4.1: now also J2.B5 (CC2)
- no-connect marks 6 -> 8
Other:
- note added: "0.1uf(100nF) = CC0805MRX7R9BB104"
- note added: "10uF = CC0805MKX5R5BB106"
- note added: "1uF = GCM219R71C105KA37D"
- note added: "22uF = C2012X5R1C226MT000E"
- note added: "2ohm = RC0805JR-072RL"
- note added: "5.1k = RC0805FR-075K1L"
- moved on the sheet: C10, FB1

Commit message: more stuff
Parts:
- removed U5: ESP32-S3-MINI-1U, symbol MCU_Espressif:ESP32-S3-MINI-1U
- added U6: ESP32-S3-MINI-1, RF_Module:ESP32-S2-MINI-1, symbol MCU_Espressif:ESP32-S3-MINI-1
- FB1: footprint (none) -> Resistor_SMD:R_0805_2012Metric_Pad1.20x1.40mm_HandSolder
Connections:
- net +3.3V: now also U6.3 (3V3)
- net ESP_32_RX: now also U6.40 (RXD0)
- net ESP_32_TX: now also U6.39 (TXD0)
- net ESP_EN: now also U6.45 (EN)
- net ESP_IO0: now also U6.4 (IO0)
- net GND: now also U6.1 (GND), U6.2 (GND), U6.42 (GND), U6.43 (GND), U6.46 (GND), U6.47 (GND), U6.48 (GND), U6.49 (GND), U6.50 (GND), U6.51 (GND), U6.52 (GND), U6.53 (GND), U6.54 (GND), U6.55 (GND), U6.56 (GND), U6.57 (GND), U6.58 (GND), U6.59 (GND), U6.60 (GND), U6.61 (GND), U6.62 (GND), U6.63 (GND), U6.64 (GND), U6.65 (GND)
Changed lines of the file:
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@@
 	)
 	(symbol
+		(lib_id "MCU_Espressif:ESP32-S3-MINI-1")
+		(at 55.88 80.01 0)
+		(unit 1)
+		(exclude_from_sim no)
+		(in_bom yes)
+		(on_board yes)
+		(dnp no)
+		(fields_autoplaced yes)
+		(property "Reference" "U6"
+			(at 58.0741 46.99 0)
+			(effects
+				(font
+					(size 1.27 1.27)
+				)
+				(justify left)
+			)
+		)
+		(property "Value" "ESP32-S3-MINI-1"
+			(at 58.0741 49.53 0)
+			(effects
+				(font
+					(size 1.27 1.27)
+				)
+				(justify left)
+			)
+		)
+		(property "Footprint" "RF_Module:ESP32-S2-MINI-1"
+			(at 55.88 77.47 0)
+			(effects
+				(font
+					(size 1.27 1.27)
+				)
+				(hide yes)
+			)
+		)
+		(property "Datasheet" "https://www.espressif.com/sites/default/files/documentation/esp32-s3-mini-1_mini-1u_datasheet_en.pdf"
+			(at 55.88 80.01 0)
+			(effects
+				(font
+					(size 1.27 1.27)
+				)
+				(hide yes)
+			)
+		)
+		(property "Description" "RF Module, ESP32-S3 SoC, Wi-Fi 802.11b/g/n, Bluetooth, BLE, 32-bit, 3.3V, SMD, onboard antenna"
+			(at 55.88 80.01 0)
+			(effects
+				(font
+					(size 1.27 1.27)
+				)
+				(hide yes)
+			)
+		)
+		(pin "33"
+		)
+		(pin "25"
+		)
+		(pin "6"
+		)
+		(pin "60"
+		)
+		(pin "16"
+		)
+		(pin "42"
+		)
+		(pin "43"
+		)
+		(pin "35"
+		)
+		(pin "3"
+		)
+		(pin "61"
+		)
+		(pin "62"
+		)
+		(pin "48"
+		)
+		(pin "23"
+		)
+		(pin "18"
+		)
+		(pin "37"
+		)
+		(pin "57"
+		)
+		(pin "63"
+		)
+		(pin "11"
+		)
+		(pin "46"
+		)
+		(pin "13"
+		)
+		(pin "54"
+		)
+		(pin "64"
+		)
+		(pin "65"
+		)
+		(pin "7"
+		)
+		(pin "8"
+		)
+		(pin "12"
+		)
+		(pin "30"
+		)
+		(pin "21"
+		)
+		(pin "47"
+		)
+		(pin "45"
+		)
+		(pin "52"
+		)
+		(pin "50"
+		)
+		(pin "15"
+		)
+		(pin "26"
+		)
+		(pin "34"
+		)
+		(pin "10"
+		)
+		(pin "19"
+		)
+		(pin "24"
+		)
+		(pin "20"
+		)
+		(pin "28"
+		)
+		(pin "29"
+		)
+		(pin "51"
+		)
+		(pin "53"
+		)
+		(pin "58"
+		)
+		(pin "56"
+		)
+		(pin "4"
+		)
+		(pin "41"
+		)
+		(pin "38"
+		)
+		(pin "49"
+		)
+		(pin "1"
+		)
+		(pin "22"
+		)
+		(pin "27"
+		)
+		(pin "31"
+		)
+		(pin "39"
+		)
+		(pin "17"
+		)
+		(pin "32"
+		)
+		(pin "5"
+		)
+		(pin "36"
+		)
+		(pin "40"
+		)
+		(pin "44"
+		)
+		(pin "55"
+		)
+		(pin "59"
+		)
+		(pin "2"
+		)
+		(pin "14"
+		)
+		(pin "9"
+		)
+		(instances
+			(project "terrarium-light"
+				(path "/15920752-a750-4c65-817e-4525ac22cfdb"
+					(reference "U6")
+					(unit 1)
+				)
+			)
+		)
+	)
+	(symbol
 		(lib_id "Device:FerriteBead_Small")
 		(at 68.58 201.93 90)
@@
 			)
 		)
-		(property "Footprint" ""
+		(property "Footprint" "Resistor_SMD:R_0805_2012Metric_Pad1.20x1.40mm_HandSolder"
 			(at 68.58 203.708 90)
 			(effects
@@
 					(unit 1)
 				)
-			)
-		)
-	)
-	(symbol
-		(lib_id "MCU_Espressif:ESP32-S3-MINI-1U")
-		(at 55.88 80.01 0)
-		(unit 1)
-		(exclude_from_sim no)
-		(in_bom yes)
-		(on_board yes)
-		(dnp no)
-		(fields_autoplaced yes)
-		(property "Reference" "U5"
-			(at 58.0741 46.99 0)
-			(effects
-				(font
-					(size 1.27 1.27)
-				)
-				(justify left)
-			)
-		)
-		(property "Value" "ESP32-S3-MINI-1U"
-			(at 58.0741 49.53 0)
-			(effects
-				(font
-					(size 1.27 1.27)
-				)
-				(justify left)
-			)
-		)
-		(property "Footprint" ""
-			(at 55.88 77.47 0)
-			(effects
-				(font
-					(size 1.27 1.27)
-				)
-				(hide yes)
-			)
-		)
-		(property "Datasheet" "https://www.espressif.com/sites/default/files/documentation/esp32-s3-mini-1_mini-1u_datasheet_en.pdf"
-			(at 55.88 80.01 0)
-			(effects
-				(font
-					(size 1.27 1.27)
-				)
-				(hide yes)
-			)
-		)
-		(property "Description" "RF Module, ESP32-S3 SoC, Wi-Fi 802.11b/g/n, Bluetooth, BLE, 32-bit, 3.3V, SMD, external antenna"
-			(at 55.88 80.01 0)
-			(effects
-				(font
-					(size 1.27 1.27)
-				)
-				(hide yes)
-			)
-		)
-		(pin "4"
-		)
-		(pin "17"
-		)
-		(pin "40"
-		)
-		(pin "41"
-		)
-		(pin "12"
-		)
-		(pin "11"
-		)
-		(pin "10"
-		)
-		(pin "18"
-		)
-		(pin "19"
-		)
-		(pin "1"
-		)
-		(pin "29"
-		)
-		(pin "3"
-		)
-		(pin "30"
-		)
-		(pin "31"
-		)
-		(pin "21"
-		)
-		(pin "22"
-		)
-		(pin "36"
-		)
-		(pin "37"
-		)
-		(pin "13"
-		)
-		(pin "44"
-		)
-		(pin "45"
-		)
-		(pin "49"
-		)
-		(pin "5"
-		)
-		(pin "50"
-		)
-		(pin "51"
-		)
-		(pin "52"
-		)
-		(pin "53"
-		)
-		(pin "54"
-		)
-		(pin "55"
-		)
-		(pin "56"
-		)
-		(pin "57"
-		)
-		(pin "58"
-		)
-		(pin "59"
-		)
-		(pin "6"
-		)
-		(pin "60"
-		)
-		(pin "61"
-		)
-		(pin "62"
-		)
-		(pin "63"
-		)
-		(pin "64"
-		)
-		(pin "65"
-		)
-		(pin "7"
-		)
-		(pin "8"
-		)
-		(pin "9"
-		)
-		(pin "2"
-		)
-		(pin "20"
-		)
-		(pin "34"
-		)
-		(pin "35"
-		)
-		(pin "23"
-		)
-		(pin "24"
-		)
-		(pin "25"
-		)
-		(pin "26"
-		)
-		(pin "32"
-		)
-		(pin "33"
-		)
-		(pin "27"
-		)
-		(pin "28"
-		)
-		(pin "38"
-		)
-		(pin "39"
-		)
-		(pin "46"
-		)
-		(pin "47"
-		)
-		(pin "48"
-		)
-		(pin "16"
-		)
-		(pin "42"
-		)
-		(pin "43"
-		)
-		(pin "15"
-		)
-		(pin "14"
-		)
-		(instances
-			(project "terrarium-light"
-				(path "/15920752-a750-4c65-817e-4525ac22cfdb"
-					(reference "U5")
-					(unit 1)
-				)

Commit message: changes
Parts:
- removed SW1: RotaryEncoder, symbol Device:RotaryEncoder
- added J1: Conn_01x04_Pin, Connector_PinHeader_2.54mm:PinHeader_1x04_P2.54mm_Vertical, symbol Connector:Conn_01x04_Pin
Connections:
- net +3.3V: now also J1.2 (Pin_2)
- net GND: now also J1.1 (Pin_1)
- new net SCL: J1.3 (Pin_3)
- new net SDA: J1.4 (Pin_4)
Changed lines of the file:
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@@
 	(wire
 		(pts
+			(xy 116.84 102.87) (xy 121.92 102.87)
+		)
+		(stroke
+			(width 0)
+			(type default)
+		)
+	)
+	(wire
+		(pts
 			(xy 163.83 251.46) (xy 177.8 251.46)
 		)
@@
 	(wire
 		(pts
+			(xy 116.84 105.41) (xy 121.92 105.41)
+		)
+		(stroke
+			(width 0)
+			(type default)
+		)
+	)
+	(wire
+		(pts
 			(xy 52.07 242.57) (xy 55.88 242.57)
 		)
@@
 		)
 	)
+	(label "SCL"
+		(at 83.82 77.47 0)
+		(fields_autoplaced yes)
+		(effects
+			(font
+				(size 1.27 1.27)
+			)
+			(justify left bottom)
+		)
+	)
 	(label "~{RTS}"
 		(at 148.59 256.54 0)
@@
 		)
 	)
+	(label "SDA"
+		(at 83.82 82.55 0)
+		(fields_autoplaced yes)
+		(effects
+			(font
+				(size 1.27 1.27)
+			)
+			(justify left bottom)
+		)
+	)
+	(label "SDA"
+		(at 116.84 102.87 0)
+		(fields_autoplaced yes)
+		(effects
+			(font
+				(size 1.27 1.27)
+			)
+			(justify left bottom)
+		)
+	)
 	(label "ESP_32_TX"
 		(at 71.12 54.61 0)
@@
 		)
 	)
+	(label "SCL"
+		(at 116.84 105.41 0)
+		(fields_autoplaced yes)
+		(effects
+			(font
+				(size 1.27 1.27)
+			)
+			(justify left bottom)
+		)
+	)
 	(label "~{DTR}"
 		(at 148.59 231.14 0)
@@
 	)
 	(symbol
-		(lib_id "Device:RotaryEncoder")
-		(at 129.54 62.23 0)
-		(unit 1)
-		(exclude_from_sim no)
-		(in_bom yes)
-		(on_board yes)
-		(dnp no)
-		(fields_autoplaced yes)
-		(property "Reference" "SW1"
-			(at 135.89 60.9599 0)
-			(effects
-				(font
-					(size 1.27 1.27)
-				)
-				(justify left)
-			)
-		)
-		(property "Value" "RotaryEncoder"
-			(at 135.89 63.4999 0)
-			(effects
-				(font
-					(size 1.27 1.27)
-				)
-				(justify left)
-			)
-		)
-		(property "Footprint" ""
-			(at 125.73 58.166 0)
-			(effects
-				(font
-					(size 1.27 1.27)
-				)
-				(hide yes)
-			)
-		)
-		(property "Datasheet" "~"
-			(at 129.54 55.626 0)
-			(effects
-				(font
-					(size 1.27 1.27)
-				)
-				(hide yes)
-			)
-		)
-		(property "Description" "Rotary encoder, dual channel, incremental quadrate outputs"
-			(at 129.54 62.23 0)
-			(effects
-				(font
-					(size 1.27 1.27)
-				)
-				(hide yes)
-			)
-		)
-		(pin "B"
-		)
-		(pin "A"
-		)
-		(pin "C"
-		)
-		(instances
-			(project "terrarium-light"
-				(path "/15920752-a750-4c65-817e-4525ac22cfdb"
-					(reference "SW1")
-					(unit 1)
-				)
-			)
-		)
-	)
-	(symbol
 		(lib_id "Device:LED")
 		(at 368.3 50.8 180)
@@
 	)
 	(symbol
+		(lib_id "power:+3.3V")
+		(at 121.92 107.95 90)
+		(unit 1)
+		(exclude_from_sim no)
+		(in_bom yes)
+		(on_board yes)
+		(dnp no)
+		(fields_autoplaced yes)
+		(property "Reference" "#PWR029"
+			(at 125.73 107.95 0)
+			(effects
+				(font
+					(size 1.27 1.27)
+				)
+				(hide yes)
+			)
+		)
+		(property "Value" "+3.3V"
+			(at 118.11 107.9499 90)
+			(effects
+				(font
+					(size 1.27 1.27)
+				)
+				(justify left)
+			)
+		)
+		(property "Footprint" ""
+			(at 121.92 107.95 0)
+			(effects
+				(font
+					(size 1.27 1.27)
+				)
+				(hide yes)
+			)
+		)
+		(property "Datasheet" ""
+			(at 121.92 107.95 0)
+			(effects
+				(font
+					(size 1.27 1.27)
+				)
+				(hide yes)
+			)
+		)
+		(property "Description" "Power symbol creates a global label with name \"+3.3V\""
+			(at 121.92 107.95 0)
+			(effects
+				(font
+					(size 1.27 1.27)
+				)
+				(hide yes)
+			)
+		)
+		(pin "1"
+		)
+		(instances
+			(project "terrarium-light"
+				(path "/15920752-a750-4c65-817e-4525ac22cfdb"
+					(reference "#PWR029")
+					(unit 1)
+				)
+			)
+		)
+	)
+	(symbol
 		(lib_id "power:GND")
 		(at 95.25 229.87 0)
@@
 	)
 	(symbol
+		(lib_id "Connector:Conn_01x04_Pin")
+		(at 127 107.95 180)
+		(unit 1)
+		(exclude_from_sim no)
+		(in_bom yes)
+		(on_board yes)
+		(dnp no)
+		(fields_autoplaced yes)
+		(property "Reference" "J1"
+			(at 128.27 105.4099 0)
+			(effects
+				(font
+					(size 1.27 1.27)
+				)
+				(justify right)
+			)
+		)
+		(property "Value" "Conn_01x04_Pin"
+			(at 128.27 107.9499 0)
+			(effects
+				(font
+					(size 1.27 1.27)
+				)
+				(justify right)
+			)
+		)
+		(property "Footprint" "Connector_PinHeader_2.54mm:PinHeader_1x04_P2.54mm_Vertical"
+			(at 127 107.95 0)
+			(effects
+				(font
+					(size 1.27 1.27)
+				)
+				(hide yes)
+			)
+		)
+		(property "Datasheet" "~"
+			(at 127 107.95 0)
+			(effects
+				(font
+					(size 1.27 1.27)
+				)
+				(hide yes)
+			)
+		)
+		(property "Description" "Generic connector, single row, 01x04, script generated"
+			(at 127 107.95 0)
+			(effects
+				(font
+					(size 1.27 1.27)
+				)
+				(hide yes)
+			)
+		)
+		(pin "3"
+		)
+		(pin "2"
+		)
+		(pin "4"
+		)
+		(pin "1"
+		)
+		(instances
+			(project "terrarium-light"
+				(path "/15920752-a750-4c65-817e-4525ac22cfdb"
+					(reference "J1")
+					(unit 1)
+				)
+			)
+		)
+	)
+	(symbol
 		(lib_id "power:VBUS")
 		(at 53.34 201.93 0)
@@
 					(unit 1)
 				)
+			)
+		)
+	)
+	(symbol
+		(lib_id "power:GND")
+		(at 121.92 110.49 0)
+		(unit 1)
+		(exclude_from_sim no)
+		(in_bom yes)
+		(on_board yes)
+		(dnp no)
+		(fields_autoplaced yes)
+		(property "Reference" "#PWR030"
+			(at 121.92 116.84 0)
+			(effects
+				(font
+					(size 1.27 1.27)
+				)
+				(hide yes)
+			)
+		)
+		(property "Value" "GND"
+			(at 121.92 115.57 0)
+			(effects
+				(font
+					(size 1.27 1.27)
+				)
+			)
+		)
+		(property "Footprint" ""
+			(at 121.92 110.49 0)
+			(effects
+				(font
+					(size 1.27 1.27)
+				)
+				(hide yes)
+			)
+		)
+		(property "Datasheet" ""
+			(at 121.92 110.49 0)
+			(effects
+				(font
+					(size 1.27 1.27)
+				)
+				(hide yes)
+			)
+		)
+		(property "Description" "Power symbol creates a global label with name \"GND\" , ground"
+			(at 121.92 110.49 0)
+			(effects
+				(font
+					(size 1.27 1.27)
+				)
+				(hide yes)
+			)
+		)
+		(pin "1"
+		)
+		(instances
+			(project "terrarium-light"
+				(path "/15920752-a750-4c65-817e-4525ac22cfdb"
+					(reference "#PWR030")
+					(unit 1)
+				)

Commit message: SO many changes
Parts:
- added C12: 0.1uF, Capacitor_SMD:C_0805_2012Metric_Pad1.18x1.45mm_HandSolder, symbol Device:C_Small
- added R5, R7, R8: 10k, Resistor_SMD:R_0805_2012Metric_Pad1.20x1.40mm_HandSolder, symbol Device:R_Small
- added R6: 1k, Resistor_SMD:R_0805_2012Metric_Pad1.20x1.40mm_HandSolder, symbol Device:R_Small
- added SW1: RotaryEncoder_Switch_MP, Rotary_Encoder:RotaryEncoder_Alps_EC12E-Switch_Vertical_H20mm_CircularMountingHoles, symbol Device:RotaryEncoder_Switch_MP
- C7: value 1uF -> 0.1uF
Connections:
- net +3.3V: now also R5.2, R7.2, R8.2
- net ESP_IO0: no longer C7.1
- net GND: now also C12.1, SW1.C, SW1.MP, SW1.S2; no longer C7.2
- new net: R5.1, R6.2, SW1.S1
- new net EncoderA: R7.1, SW1.A
- new net EncoderB: R8.1, SW1.B
- new net EncoderButton: C12.2, R6.1

Commit message: saving
Connections:
- net +3.3V: now also C7.2
- net GND: now also C7.1
Other:
- moved on the sheet: C7
Changed lines of the file:
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@@
 	)
 	(junction
+		(at 111.76 107.95)
+		(diameter 0)
+		(color 0 0 0 0)
+	)
+	(junction
 		(at 271.78 114.3)
 		(diameter 0)
@@
 	(wire
 		(pts
+			(xy 111.76 107.95) (xy 121.92 107.95)
+		)
+		(stroke
+			(width 0)
+			(type default)
+		)
+	)
+	(wire
+		(pts
 			(xy 215.9 114.3) (xy 228.6 114.3)
 		)
@@
 	(wire
 		(pts
+			(xy 110.49 107.95) (xy 111.76 107.95)
+		)
+		(stroke
+			(width 0)
+			(type default)
+		)
+	)
+	(wire
+		(pts
 			(xy 215.9 50.8) (xy 228.6 50.8)
 		)
@@
 	(symbol
 		(lib_id "Device:C_Small")
-		(at 113.03 115.57 90)
+		(at 111.76 110.49 180)
 		(unit 1)
 		(exclude_from_sim no)
@@
 		(fields_autoplaced yes)
 		(property "Reference" "C7"
-			(at 113.0363 109.22 90)
+			(at 114.3 109.2135 0)
 			(effects
 				(font
 					(size 1.27 1.27)
 				)
+				(justify right)
 			)
 		)
 		(property "Value" "0.1uF "
-			(at 113.0363 111.76 90)
+			(at 114.3 111.7535 0)
 			(effects
 				(font
 					(size 1.27 1.27)
 				)
+				(justify right)
 			)
 		)
 		(property "Footprint" "Capacitor_SMD:C_0805_2012Metric_Pad1.18x1.45mm_HandSolder"
-			(at 113.03 115.57 0)
+			(at 111.76 110.49 0)
 			(effects
 				(font
@@
 		)
 		(property "Datasheet" "~"
-			(at 113.03 115.57 0)
+			(at 111.76 110.49 0)
 			(effects
 				(font
@@
 		)
 		(property "Description" "Unpolarized capacitor, small symbol"
-			(at 113.03 115.57 0)
+			(at 111.76 110.49 0)
 			(effects
 				(font
@@
 	(symbol
 		(lib_id "power:+3.3V")
-		(at 121.92 107.95 90)
+		(at 110.49 107.95 90)
 		(unit 1)
 		(exclude_from_sim no)
@@
 		(fields_autoplaced yes)
 		(property "Reference" "#PWR029"
-			(at 125.73 107.95 0)
+			(at 114.3 107.95 0)
 			(effects
 				(font
@@
 		)
 		(property "Value" "+3.3V"
-			(at 118.11 107.9499 90)
+			(at 106.68 107.9499 90)
 			(effects
 				(font
@@
 		)
 		(property "Footprint" ""
-			(at 121.92 107.95 0)
+			(at 110.49 107.95 0)
 			(effects
 				(font
@@
 		)
 		(property "Datasheet" ""
-			(at 121.92 107.95 0)
+			(at 110.49 107.95 0)
 			(effects
 				(font
@@
 		)
 		(property "Description" "Power symbol creates a global label with name \"+3.3V\""
-			(at 121.92 107.95 0)
+			(at 110.49 107.95 0)
 			(effects
 				(font
@@
 					(unit 1)
 				)
+			)
+		)
+	)
+	(symbol
+		(lib_id "power:GND")
+		(at 111.76 113.03 0)
+		(unit 1)
+		(exclude_from_sim no)
+		(in_bom yes)
+		(on_board yes)
+		(dnp no)
+		(fields_autoplaced yes)
+		(property "Reference" "#PWR036"
+			(at 111.76 119.38 0)
+			(effects
+				(font
+					(size 1.27 1.27)
+				)
+				(hide yes)
+			)
+		)
+		(property "Value" "GND"
+			(at 111.76 118.11 0)
+			(effects
+				(font
+					(size 1.27 1.27)
+				)
+			)
+		)
+		(property "Footprint" ""
+			(at 111.76 113.03 0)
+			(effects
+				(font
+					(size 1.27 1.27)
+				)
+				(hide yes)
+			)
+		)
+		(property "Datasheet" ""
+			(at 111.76 113.03 0)
+			(effects
+				(font
+					(size 1.27 1.27)
+				)
+				(hide yes)
+			)
+		)
+		(property "Description" "Power symbol creates a global label with name \"GND\" , ground"
+			(at 111.76 113.03 0)
+			(effects
+				(font
+					(size 1.27 1.27)
+				)
+				(hide yes)
+			)
+		)
+		(pin "1"
+		)
+		(instances
+			(project "terrarium-light"
+				(path "/15920752-a750-4c65-817e-4525ac22cfdb"
+					(reference "#PWR036")
+					(unit 1)
+				)

Commit message: settings
Parts:
- C12, C5, C6, C7: value 0.1uF -> 0.1uF
Connections:
- no-connect marks 8 -> 14
Changed lines of the file:
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@@
 	)
 	(no_connect
+		(at 40.64 77.47)
+	)
+	(no_connect
+		(at 40.64 82.55)
+	)
+	(no_connect
 		(at 120.65 251.46)
 	)
 	(no_connect
+		(at 40.64 87.63)
+	)
+	(no_connect
+		(at 40.64 85.09)
+	)
+	(no_connect
 		(at 120.65 248.92)
 	)
@@
 	)
 	(no_connect
+		(at 40.64 80.01)
+	)
+	(no_connect
 		(at 52.07 257.81)
 	)
@@
 		(at 120.65 246.38)
 	)
+	(no_connect
+		(at 40.64 74.93)
+	)
 	(wire
 		(pts
@@
 	(wire
 		(pts
+			(xy 71.12 67.31) (xy 73.66 67.31)
+		)
+		(stroke
+			(width 0)
+			(type default)
+		)
+	)
+	(wire
+		(pts
 			(xy 158.75 50.8) (xy 167.64 50.8)
 		)
@@
 	(wire
 		(pts
+			(xy 71.12 69.85) (xy 73.66 69.85)
+		)
+		(stroke
+			(width 0)
+			(type default)
+		)
+	)
+	(wire
+		(pts
 			(xy 181.61 50.8) (xy 181.61 54.61)
 		)
@@
 		)
 	)
+	(label "EncoderB"
+		(at 97.79 83.82 0)
+		(fields_autoplaced yes)
+		(effects
+			(font
+				(size 1.27 1.27)
+			)
+			(justify left bottom)
+		)
+	)
+	(label "EncoderA"
+		(at 93.98 91.44 0)
+		(fields_autoplaced yes)
+		(effects
+			(font
+				(size 1.27 1.27)
+			)
+			(justify left bottom)
+		)
+	)
 	(label "D+"
 		(at 55.88 246.38 0)
@@
 		)
 	)
+	(label "EncoderButton"
+		(at 109.22 78.74 0)
+		(fields_autoplaced yes)
+		(effects
+			(font
+				(size 1.27 1.27)
+			)
+			(justify left bottom)
+		)
+	)
 	(label "D+"
 		(at 96.52 243.84 0)
@@
 			)
 		)
-		(property "Value" "0.1uF "
+		(property "Value" "0.1uF"
 			(at 105.4163 226.06 90)
 			(effects
@@
 			)
 		)
-		(property "Value" "0.1uF "
+		(property "Value" "0.1uF"
 			(at 114.3 111.7535 0)
 			(effects
@@
 			)
 		)
-		(property "Value" "0.1uF "
+		(property "Value" "0.1uF"
 			(at 113.0363 226.06 90)
 			(effects
@@
 			)
 		)
-		(property "Value" "0.1uF "
+		(property "Value" "0.1uF"
 			(at 184.15 58.4135 0)
 			(effects
